File: PCBs/DisplayPruebas/DisplayTestBoard.brd (EAGLE design)
At the start: 100 x 50 mm, 41 parts, among them CN1 LPPB052NFSS-RC, CN2 01-014-0371, IC2 01-012-0185, K2 01-015-0021, Q1 01-041-0013

Commit message: Repository Clean Up
Se hace limpieza de repositorio
Parts:
- removed C25: 01-009-0145, PegasusControl:CT3528
- removed CN1: LPPB052NFSS-RC, PegasusControl:2X5_0.1_SMD_BE
- added JTAG: SAMTECSTR2X5, troyaIII:SAMTECSTR2X5
- C20: value 01-009-0105 -> 01-009-0145
- R3: value ERJ-6GEYJ103V -> 10K
- moved Q1 141.9 mm to (64.5, 14.4), turned to 180 degrees
- moved C10 134.7 mm to (60.8, 31.0)
- moved K2 131.8 mm to (63.4, 10.0), turned to 180 degrees
- moved R4 130.7 mm to (56.8, 37.9), turned to 180 degrees
- moved C9 126.1 mm to (60.8, 24.0)
- moved C14 123.1 mm to (58.1, 5.19), turned to 180 degrees
- moved C3 122.0 mm to (39.0, 22.1), turned to 180 degrees
- moved C16 119.1 mm to (56.8, 40.0)
- moved R1 117.5 mm to (40.5, 14.5)
- moved C8 114.3 mm to (54.1, 13.0), turned to 180 degrees
- moved C19 114.1 mm to (67.0, 34.5)
- moved D2 113.0 mm to (44.2, 14.5)
- moved C2 110.5 mm to (39.0, 24.2), turned to 180 degrees
- moved C13 109.1 mm to (58.1, 3.09), turned to 180 degrees
- moved R5 107.8 mm to (64.4, 18.0)
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Connections:
- removed net DISP_C3+: C19.+, CN2.17
- removed net DISP_D/C: CN2.3, IC1.96
- new net DISP_A0: CN2.3, IC1.77
- new net DISP_RD: CN2.5, IC1.79
- new net DISP_WR: CN2.4, IC1.78
- net +3V3: now also JTAG.P$1, R3.2; no longer CN1.1, CN2.30, CN2.4, CN2.5, R3.1
- net DISP_BL: now also IC1.54; no longer IC1.98
- net DISP_C1+: now also C19.+; no longer C20.+
- net DISP_C1-: no longer C20.-
- net DISP_RESET: now also IC1.76; no longer IC1.97
- net DISP_V0: now also C24.+; no longer C25.+
- net DISP_V1: now also C23.+, CN2.25; no longer C21.+, CN2.22
- net DISP_V2: now also CN2.24; no longer CN2.23
- net DISP_V3: now also C21.+, CN2.23; no longer C23.+, CN2.24
- net DISP_V4: now also C20.+, CN2.22; no longer C24.+, CN2.25
- net DISP_VOUT: now also CN2.17
- net GND: now also C20.-, CN2.30, JTAG.P$2, JTAG.P$3; no longer C25.-, CN1.3, CN1.5
- net JTAG_TCLK: now also JTAG.P$7; no longer CN1.4
- net JTAG_TDI: now also JTAG.P$9; no longer CN1.8
- net JTAG_TDO: now also JTAG.P$8; no longer CN1.6
- net JTAG_TMS: now also JTAG.P$6, R3.1; no longer CN1.2, R3.2
- net LED: now also IC1.33; no longer IC1.79
- net RESET: now also JTAG.P$10; no longer CN1.10
Routing:
- net +3V3: track 0.00 -> 30.6 mm
- net DISP_V0: track 0.00 -> 25.5 mm, vias 0 -> 1
- net DISP_V1: track 0.00 -> 24.4 mm, vias 0 -> 1
- net RESET: track 0.00 -> 24.2 mm, vias 0 -> 2
- net XTAL: track 0.00 -> 23.8 mm
- net DISP_V2: track 0.00 -> 21.9 mm, vias 0 -> 1
- net JTAG_TMS: track 0.00 -> 21.5 mm, vias 0 -> 2
- net VMAIN: track 0.00 -> 21.0 mm
- net DISP_V3: track 0.00 -> 19.9 mm, vias 0 -> 1
- net N$21: track 0.00 -> 17.7 mm
- net DISP_WR: track 0.00 -> 16.5 mm, vias 0 -> 1
- net JTAG_TDI: track 0.00 -> 15.4 mm, vias 0 -> 2
- net DISP_SDO: track 0.00 -> 14.7 mm, vias 0 -> 1
- net DISP_CLK: track 0.00 -> 14.2 mm, vias 0 -> 1
- net EXTAL: track 0.00 -> 14.1 mm
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