File: PCBs/DisplayPruebas/DisplayTestBoard.sch (EAGLE design)
At the start: 41 parts, among them CN1 LPPB052NFSS-RC, CN2 01-014-0371, IC2 01-012-0185, K2 01-015-0021, Q1 01-041-0013

Commit message: Repository Clean Up
Se hace limpieza de repositorio
Parts:
- removed C25: 01-009-0145, PegasusControl:01-009-0145
- removed CN1: LPPB052NFSS-RC, PegasusControl:LPPB052NFSS-RC
- added JTAG: SAMTECSTR2X5, troyaIII:SAMTECSTR2X5
- C20: value 01-009-0105 -> 01-009-0145; device PegasusControl:01-009-0105 -> PegasusControl:01-009-0145
- R3: value ERJ-6GEYJ103V -> 10K; device PegasusControl:ERJ-6GEYJ103V -> PegasusControl:01-030-0334
Connections:
- removed net DISP_C3+: C19.+, CN2.C3+
- removed net DISP_D/C: CN2.A0, IC1.PTD3
- new net DISP_A0: CN2.A0, IC1.PTC5
- new net DISP_RD: CN2./RD, IC1.PTC7
- new net DISP_WR: CN2./WR, IC1.PTC6
- net +3V3: now also JTAG.1, R3.2; no longer CN1.1, CN2./RD, CN2./WR, CN2.IRS, R3.1
- net DISP_BL: now also IC1.PTB1; no longer IC1.PTD5
- net DISP_C1+: now also C19.+; no longer C20.+
- net DISP_C1-: no longer C20.-
- net DISP_RESET: now also IC1.PTC4; no longer IC1.PTD4
- net DISP_V0: now also C24.+; no longer C25.+
- net DISP_V1: now also C23.+; no longer C21.+
- net DISP_V3: now also C21.+; no longer C23.+
- net DISP_V4: now also C20.+; no longer C24.+
- net DISP_VOUT: now also CN2.C3+
- net GND: now also C20.-, CN2.NC, JTAG.3, JTAG.5; no longer C25.-, CN1.3, CN1.5
- net JTAG_TCLK: now also JTAG.4; no longer CN1.4
- net JTAG_TDI: now also JTAG.8; no longer CN1.8
- net JTAG_TDO: now also JTAG.6; no longer CN1.6
- net JTAG_TMS: now also JTAG.2, R3.1; no longer CN1.2, R3.2
- net LED: now also IC1.PTE26; no longer IC1.PTC7
- net RESET: now also JTAG.10; no longer CN1.10
Other:
- moved on the sheet: C20, C21, C22, C23, C24, R3
